File: scratch/waferspace_cob/waferspace_cob/waferspace_cob.kicad_sch (KiCad schematic)
At the start: 11 parts, among them J101 Conn_01x12, J102 Conn_01x12, J103 Conn_01x12, J104 Conn_01x12, J105 Conn_01x20, J106 Conn_01x20, U101 Caravel_COB, U102 Caravel_COB

Commit message: padring v0.1
Parts:
- U102: footprint WafeSpace:caravel_gfmpw_1_0_asap -> WafeSpace:waferspace_default_padring_v0
Changed lines of the file:
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@@
 			)
 		)
-		(property "Footprint" "WafeSpace:caravel_gfmpw_1_0_asap"
+		(property "Footprint" "WafeSpace:waferspace_default_padring_v0"
 			(at 223.52 93.98 0)
 			(effects
