File: 74pad-70pin-mezzanine/74pad-70pin-mezzanine.kicad_sch (KiCad schematic)
At the start: 11 parts

Commit message: fix and add project code areas to panel
Parts:
- C101, C102, C103, C104, C105, C106, C107, C108: value C_Small -> 1 uF
- U101: value ~ -> (none); footprint Connector_Mezzanine:CONN-SMD_70P-P0.40_HCTL_HC-PBB40C-70DP-0.4V-02 -> Connector:CONN-SMD_70P-P0.40_HCTL_HC-PBB40C-70DP-0.4V-02
- U102: value ~ -> (none); now not fitted; now left out of the parts list
- U2: value ~ -> (none)
