File: mezzanine-1x0p5/mezzanine-1x0p5.kicad_pcb (KiCad board)
At the start: 2 copper layers, 14 x 16 mm, 11 parts

Commit message: 1x0p5 routed
Connections:
- U101 pad 12: /bidir_45 -> /in_0
- U101 pad 13: /bidir_44 -> /in_1
- U101 pad 14: /bidir_43 -> /in_2
- U101 pad 15: /bidir_42 -> /in_3
- U101 pad 16: /bidir_41 -> /an_3
- U101 pad 17: /bidir_40 -> /an_2
- U101 pad 20: /an_3 -> /an_1
- U101 pad 21: /an_2 -> /an_0
- U101 pad 22: /in_3 -> /bidir_45
- U101 pad 23: /in_2 -> /bidir_44
- U101 pad 26: /in_1 -> /bidir_43
- U101 pad 27: /in_0 -> /bidir_42
- U101 pad 28: /an_1 -> /bidir_41
- U101 pad 29: /an_0 -> /bidir_40
Routing:
- net GND: track 6.55 -> 55.3 mm, vias 32 -> 30
- net VDD_IO_2: track 0.00 -> 12.7 mm
- net /bidir_41: track 0.00 -> 10.6 mm
- net /bidir_40: track 0.00 -> 10.0 mm, vias 0 -> 1
- net PWR_AUX_1: track 0.00 -> 8.30 mm, vias 0 -> 1
- net /in_0: track 0.00 -> 8.10 mm
- net /bidir_45: track 0.00 -> 7.18 mm, vias 0 -> 1
- net /bidir_42: track 0.00 -> 6.84 mm
- net /in_1: track 0.00 -> 6.76 mm
- net /bidir_43: track 0.00 -> 6.24 mm, vias 0 -> 1
- net /an_2: track 0.00 -> 5.63 mm, vias 0 -> 1
- net /in_2: track 0.00 -> 4.97 mm
- net /an_1: track 0.00 -> 4.76 mm
- net /bidir_44: track 0.00 -> 3.65 mm, vias 0 -> 1
- net /an_3: track 0.00 -> 3.43 mm, vias 0 -> 1
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Other:
- board text added: "70 PIN MEZZANINE 72 PIN PADRING VERSION: 1x0p5"
- board text removed: "70 PIN MEZZANINE 74 PIN PADRING VERSION: TT01"
