File: mezzanine-1x0p5/mezzanine-1x0p5.kicad_sch (KiCad schematic)
At the start: 10 parts

Commit message: 1x0p5 routed
Parts:
- U101, U102: value ~ -> (none)
Connections:
- net an_0: now also U101.21 (in_4); no longer U101.29 (an_0)
- net an_1: now also U101.20 (in_5); no longer U101.28 (an_1)
- net an_2: now also U101.17 (in_6); no longer U101.21 (in_4)
- net an_3: now also U101.16 (in_7); no longer U101.20 (in_5)
- net bidir_40: now also U101.29 (an_0); no longer U101.17 (in_6)
- net bidir_41: now also U101.28 (an_1); no longer U101.16 (in_7)
- net bidir_42: now also U101.27 (in_0); no longer U101.15 (in_8)
- net bidir_43: now also U101.26 (in_1); no longer U101.14 (in_9)
- net bidir_44: now also U101.23 (in_2); no longer U101.13 (in_10)
- net bidir_45: now also U101.22 (in_3); no longer U101.12 (in_11)
- net in_0: now also U101.12 (in_11); no longer U101.27 (in_0)
- net in_1: now also U101.13 (in_10); no longer U101.26 (in_1)
- net in_2: now also U101.14 (in_9); no longer U101.23 (in_2)
- net in_3: now also U101.15 (in_8); no longer U101.22 (in_3)
