File: mezzanine-0p5x1/mezzanine-0p5x1.kicad_pcb (KiCad board)
At the start: 2 copper layers, 14 x 16 mm, 1 part

Commit message: WIP 0p5x1 - probably need to try again
Parts:
- removed U1: ~, WaferSpace:waferspace_p5x1_padring_v0.2
- added C101: C_Small, Capacitor_SMD:C_0201_0603Metric, B.Cu at (93.5, 105.4)
- added C102: C_Small, Capacitor_SMD:C_0201_0603Metric, B.Cu at (106.0, 94.7)
- added C103: C_Small, Capacitor_SMD:C_0201_0603Metric, B.Cu at (93.5, 103.1)
- added C104: C_Small, Capacitor_SMD:C_0201_0603Metric, B.Cu at (106.0, 97.2)
- added C105: C_Small, Capacitor_SMD:C_0201_0603Metric, B.Cu at (93.5, 99.8)
- added C106: C_Small, Capacitor_SMD:C_0201_0603Metric, B.Cu at (106.0, 99.8)
- added C107: C_Small, Capacitor_SMD:C_0201_0603Metric, B.Cu at (93.5, 95.0)
- added C108: C_Small, Capacitor_SMD:C_0201_0603Metric, B.Cu at (106.0, 101.7)
- added G***: LOGO, Symbol:waferspace_pin1_silk, F.Cu at (104.5, 93.5)
- added U101: ~, WaferSpace:CONN-SMD_70P-P0.40_HCTL_HC-PBB40C-70DP-0.4V-02, B.Cu at (99.8, 99.8)
- added U102: ~, WaferSpace:waferspace_p5x1_padring_v0.2, F.Cu at (99.8, 99.9)
Routing:
- net GND: track 0.00 -> 43.0 mm, vias 0 -> 26
- net /an_4: track 0.00 -> 25.8 mm, vias 0 -> 1
- net /an_5: track 0.00 -> 23.9 mm, vias 0 -> 1
- net VDD_CORE_0: track 0.00 -> 9.81 mm, vias 0 -> 1
- net PWR_AUX_0: track 0.00 -> 9.43 mm, vias 0 -> 1
- net VDD_IO_2: track 0.00 -> 8.34 mm, vias 0 -> 3
- net VDD_IO_1: track 0.00 -> 8.31 mm, vias 0 -> 1
- net /bidir_20: track 0.00 -> 7.60 mm, vias 0 -> 1
- net /bidir_42: track 0.00 -> 7.36 mm, vias 0 -> 1
- net /bidir_41: track 0.00 -> 7.22 mm, vias 0 -> 1
- net /bidir_40: track 0.00 -> 7.19 mm, vias 0 -> 1
- net /bidir_19: track 0.00 -> 7.16 mm, vias 0 -> 1
- net /bidir_39: track 0.00 -> 6.50 mm, vias 0 -> 1
- net /bidir_28: track 0.00 -> 6.30 mm, vias 0 -> 1
- net /bidir_21: track 0.00 -> 6.25 mm, vias 0 -> 1
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- added copper zone on B.Cu, net GND
- added copper zone on F.Cu, net GND
Other:
- board text added: "70 PIN MEZZANINE 72 PIN PADRING VERSION: 1x0p5"
- board text added: "Allocated Space For Passives"
- board text added: "wafer.space GF180MCU Run 1"

Commit message: Diagonal die
Parts:
- moved C103 1.01 mm to (94.5, 103.1)
- moved C101 0.99 mm to (94.5, 105.5)
- moved C108 0.45 mm to (106.0, 102.1), turned to -90 degrees
- turned C106 to 90 degrees
- turned U102 to -45 degrees
Connections:
- U101 pad 12: /an_0 -> /in_3
- U101 pad 13: /an_1 -> /in_2
- U101 pad 14: /an_2 -> /bidir_43
- U101 pad 15: /an_3 -> /bidir_42
- U101 pad 16: /in_3 -> /bidir_41
- U101 pad 17: /in_2 -> /bidir_40
- U101 pad 20: /an_4 -> /bidir_39
- U101 pad 21: /an_5 -> /bidir_38
- U101 pad 22: /bidir_43 -> /bidir_37
- U101 pad 23: /bidir_42 -> /bidir_36
- U101 pad 28: /bidir_41 -> /bidir_35
- U101 pad 29: /bidir_40 -> /bidir_34
- U101 pad 30: /bidir_39 -> /bidir_33
- U101 pad 31: /bidir_38 -> /bidir_32
- U101 pad 32: /bidir_37 -> /bidir_31
- U101 pad 33: /bidir_36 -> /bidir_30
- U101 pad 34: /bidir_35 -> /bidir_29
- U101 pad 35: /bidir_34 -> /bidir_28
- U101 pad 36: /bidir_33 -> /an_5
- U101 pad 37: /bidir_32 -> /an_4
- U101 pad 38: /bidir_31 -> /an_3
- U101 pad 39: /bidir_30 -> /an_2
- U101 pad 40: /bidir_29 -> /an_1
- U101 pad 41: /bidir_28 -> /an_0
Routing:
- net /an_5: track 23.9 -> 3.67 mm
- net /an_4: track 25.8 -> 5.53 mm
- net /in_1: track 0.00 -> 17.0 mm, vias 0 -> 1
- net /in_0: track 0.00 -> 16.6 mm
- net /bidir_24: track 3.45 -> 16.1 mm
- net VDD_IO_3: track 0.00 -> 11.4 mm, vias 1 -> 2
- net /bidir_23: track 5.21 -> 16.3 mm
- net /bidir_22: track 5.84 -> 16.4 mm
- net PWR_AUX_0: track 9.43 -> 0.00 mm
- net /bidir_3: track 0.00 -> 8.91 mm
- net PWR_AUX_1: track 0.00 -> 8.91 mm
- net /bidir_2: track 0.00 -> 8.47 mm
- net VDD_CORE_1: track 0.00 -> 8.25 mm, vias 1 -> 2
- net /rst_n: track 0.00 -> 7.97 mm
- net /bidir_4: track 0.00 -> 7.81 mm
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