File: mezzanine-0p5x1/mezzanine-0p5x1.kicad_sch (KiCad schematic)
At the start: 2 parts

Commit message: create p5x1 padring
Parts:
- U1: value ~ -> (none); footprint (none) -> WaferSpace:waferspace_p5x1_padring_v0.2
- U101: value ~ -> (none)
Other:
- moved on the sheet: U1
Changed lines of the file:
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@@
 (kicad_sch
-	(version 20250114)
+	(version 20260306)
 	(generator "eeschema")
-	(generator_version "9.0")
+	(generator_version "10.0")
 	(paper "A4")
 	(junction
@@
 		(at 44.45 146.05 0)
 		(unit 1)
+		(body_style 1)
 		(exclude_from_sim no)
 		(in_bom yes)
 		(on_board yes)
+		(in_pos_files yes)
 		(dnp no)
 		(fields_autoplaced yes)
 		(property "Reference" "#PWR02"
 			(at 44.45 152.4 0)
-			(effects
-				(font
-					(size 1.27 1.27)
-				)
-				(hide yes)
+			(hide yes)
+			(show_name no)
+			(do_not_autoplace no)
+			(effects
+				(font
+					(size 1.27 1.27)
+				)
 			)
 		)
 		(property "Value" "GND"
 			(at 44.45 151.13 0)
+			(show_name no)
+			(do_not_autoplace no)
 			(effects
 				(font
@@
 		(property "Footprint" ""
 			(at 44.45 146.05 0)
-			(effects
-				(font
-					(size 1.27 1.27)
-				)
-				(hide yes)
+			(hide yes)
+			(show_name no)
+			(do_not_autoplace no)
+			(effects
+				(font
+					(size 1.27 1.27)
+				)
 			)
 		)
 		(property "Datasheet" ""
 			(at 44.45 146.05 0)
-			(effects
-				(font
-					(size 1.27 1.27)
-				)
-				(hide yes)
+			(hide yes)
+			(show_name no)
+			(do_not_autoplace no)
+			(effects
+				(font
+					(size 1.27 1.27)
+				)
 			)
 		)
 		(property "Description" "Power symbol creates a global label with name \"GND\" , ground"
 			(at 44.45 146.05 0)
-			(effects
-				(font
-					(size 1.27 1.27)
-				)
-				(hide yes)
+			(hide yes)
+			(show_name no)
+			(do_not_autoplace no)
+			(effects
+				(font
+					(size 1.27 1.27)
+				)
 			)
 		)
@@
 	(symbol
 		(lib_id "WaferSpace:0p5x1")
-		(at 163.83 110.49 0)
+		(at 163.83 54.61 270)
 		(unit 1)
+		(body_style 1)
 		(exclude_from_sim no)
 		(in_bom yes)
 		(on_board yes)
+		(in_pos_files yes)
 		(dnp no)
 		(fields_autoplaced yes)
 		(property "Reference" "U1"
-			(at 245.11 71.0498 0)
-			(effects
-				(font
-					(size 1.27 1.27)
-				)
-			)
-		)
-		(property "Value" "~"
-			(at 245.11 73.5898 0)
-			(effects
-				(font
-					(size 1.27 1.27)
-				)
-			)
-		)
-		(property "Footprint" ""
-			(at 163.83 110.49 0)
-			(effects
-				(font
-					(size 1.27 1.27)
-				)
-				(hide yes)
+			(at 199.9681 41.91 90)
+			(show_name no)
+			(do_not_autoplace no)
+			(effects
+				(font
+					(size 1.27 1.27)
+				)
+				(justify left)
+			)
+		)
+		(property "Value" ""
+			(at 200.7302 135.89 0)
+			(show_name no)
+			(do_not_autoplace no)
+			(effects
+				(font
+					(size 1.27 1.27)
+				)
+			)
+		)
+		(property "Footprint" "WaferSpace:waferspace_p5x1_padring_v0.2"
+			(at 163.83 54.61 0)
+			(hide yes)
+			(show_name no)
+			(do_not_autoplace no)
+			(effects
+				(font
+					(size 1.27 1.27)
+				)
 			)
 		)
 		(property "Datasheet" ""
-			(at 163.83 110.49 0)
-			(effects
-				(font
-					(size 1.27 1.27)
-				)
-				(hide yes)
+			(at 163.83 54.61 0)
+			(hide yes)
+			(show_name no)
+			(do_not_autoplace no)
+			(effects
+				(font
+					(size 1.27 1.27)
+				)
 			)
 		)
 		(property "Description" ""
-			(at 163.83 110.49 0)
-			(effects
-				(font
-					(size 1.27 1.27)
-				)
-				(hide yes)
+			(at 163.83 54.61 0)
+			(hide yes)
+			(show_name no)
+			(do_not_autoplace no)
+			(effects
+				(font
+					(size 1.27 1.27)
+				)
 			)
 		)
@@
 		)
 		(instances
-			(project ""
+			(project "mezzanine-0p5x1"
 				(path "/3496b536-e2ac-465d-a0f3-b91c8ceb317b"
 					(reference "U1")
@@
 		(at 77.47 88.9 0)
 		(unit 1)
+		(body_style 1)
 		(exclude_from_sim no)
 		(in_bom yes)
 		(on_board yes)
+		(in_pos_files yes)
 		(dnp no)
 		(property "Reference" "U101"
 			(at 92.71 82.55 0)
+			(show_name no)
+			(do_not_autoplace no)
 			(effects
 				(font
@@
 			)
 		)
-		(property "Value" "~"
+		(property "Value" ""
 			(at 95.25 123.19 0)
+			(show_name no)
+			(do_not_autoplace no)
 			(effects
 				(font
@@
 		(property "Footprint" "WaferSpace:CONN-SMD_70P-P0.40_HCTL_HC-PBB40C-70DP-0.4V-02"
 			(at 78.232 77.978 0)
-			(effects
-				(font
-					(size 1.27 1.27)
-				)
-				(hide yes)
+			(hide yes)
+			(show_name no)
+			(do_not_autoplace no)
+			(effects
+				(font
+					(size 1.27 1.27)
+				)
 			)
 		)
 		(property "Datasheet" ""
 			(at 77.47 88.9 0)
-			(effects
-				(font
-					(size 1.27 1.27)
-				)
-				(hide yes)
+			(hide yes)
+			(show_name no)
+			(do_not_autoplace no)
+			(effects
+				(font
+					(size 1.27 1.27)
+				)
 			)
 		)
 		(property "Description" ""
 			(at 77.47 88.9 0)
-			(effects
-				(font
-					(size 1.27 1.27)
-				)
-				(hide yes)
+			(hide yes)
+			(show_name no)
+			(do_not_autoplace no)
+			(effects
+				(font
+					(size 1.27 1.27)
+				)
 			)
 		)
@@
 		(at 114.3 146.05 0)
 		(unit 1)
+		(body_style 1)
 		(exclude_from_sim no)
 		(in_bom yes)
 		(on_board yes)
+		(in_pos_files yes)
 		(dnp no)
 		(fields_autoplaced yes)
 		(property "Reference" "#PWR01"
 			(at 114.3 152.4 0)
-			(effects
-				(font
-					(size 1.27 1.27)
-				)
-				(hide yes)
+			(hide yes)
+			(show_name no)
+			(do_not_autoplace no)
+			(effects
+				(font
+					(size 1.27 1.27)
+				)
 			)
 		)
 		(property "Value" "GND"
 			(at 114.3 151.13 0)
+			(show_name no)
+			(do_not_autoplace no)
 			(effects
 				(font
@@
 		(property "Footprint" ""
 			(at 114.3 146.05 0)
-			(effects
-				(font
-					(size 1.27 1.27)
-				)
-				(hide yes)
+			(hide yes)
+			(show_name no)
+			(do_not_autoplace no)
+			(effects
+				(font
+					(size 1.27 1.27)
+				)
 			)
 		)
 		(property "Datasheet" ""
 			(at 114.3 146.05 0)
-			(effects
-				(font
-					(size 1.27 1.27)
-				)
-				(hide yes)
+			(hide yes)
+			(show_name no)
+			(do_not_autoplace no)
+			(effects
+				(font
+					(size 1.27 1.27)
+				)
 			)
 		)
 		(property "Description" "Power symbol creates a global label with name \"GND\" , ground"
 			(at 114.3 146.05 0)
-			(effects
-				(font
-					(size 1.27 1.27)
-				)
-				(hide yes)
+			(hide yes)
+			(show_name no)
+			(do_not_autoplace no)
+			(effects
+				(font
+					(size 1.27 1.27)
+				)
 			)
 		)
@@
 		(at 81.28 138.43 0)
 		(unit 1)
+		(body_style 1)
 		(exclude_from_sim no)
 		(in_bom yes)
 		(on_board yes)
+		(in_pos_files yes)
 		(dnp no)
 		(fields_autoplaced yes)
 		(property "Reference" "#PWR03"
 			(at 81.28 144.78 0)
-			(effects
-				(font
-					(size 1.27 1.27)
-				)
-				(hide yes)
+			(hide yes)
+			(show_name no)
+			(do_not_autoplace no)
+			(effects
+				(font
+					(size 1.27 1.27)
+				)
 			)
 		)
 		(property "Value" "GND"
 			(at 81.28 143.51 0)
+			(show_name no)
+			(do_not_autoplace no)
 			(effects
 				(font
@@
 		(property "Footprint" ""
 			(at 81.28 138.43 0)
-			(effects
-				(font
-					(size 1.27 1.27)
-				)
-				(hide yes)
+			(hide yes)
+			(show_name no)
+			(do_not_autoplace no)
+			(effects
+				(font
+					(size 1.27 1.27)
+				)
 			)
 		)
 		(property "Datasheet" ""
 			(at 81.28 138.43 0)
-			(effects
-				(font
-					(size 1.27 1.27)
-				)
-				(hide yes)
+			(hide yes)
+			(show_name no)
+			(do_not_autoplace no)
+			(effects
+				(font
+					(size 1.27 1.27)
+				)
 			)
 		)
 		(property "Description" "Power symbol creates a global label with name \"GND\" , ground"
 			(at 81.28 138.43 0)
-			(effects
-				(font
-					(size 1.27 1.27)
-				)
-				(hide yes)
-			)
-		)
+			(hide yes)
+			(show_name no)
+			(do_not_autoplace no)
+			(effects
+				(font
+					(size 1.27 1.27)
+				)
+			)
+		)

Commit message: WIP 0p5x1 - probably need to try again
Parts:
- added C101, C102, C103, C104, C105, C106, C107, C108: C_Small, Capacitor_SMD:C_0201_0603Metric, symbol Device:C_Small
- renumbered U1 to U102
Connections:
- net bidir_44 is gone; now on net an_1: U101.13 (in_10)
- net bidir_45 is gone; now on net an_0: U101.12 (in_11)
- net GND: now also U102.14 (GND), U102.23 (GND), U102.3 (GND), U102.33 (GND), U102.42 (GND), U102.51 (GND), U102.61 (GND), U102.68 (GND), U102.75 (MP), U102.76 (MP), U102.77 (MP), U102.78 (MP), U102.79 (MP), U102.80 (MP), U102.81 (MP), C101.2, C102.2, C103.2, C104.2, C105.2, C106.2, C107.2, C108.2
- net PWR_AUX_0: now also U102.24 (VDD), C105.1
- net PWR_AUX_1: now also U102.60 (VDD), C106.1
- net VDD_CORE_0: now also U102.32 (VDD), C103.1
- net VDD_CORE_1: now also U102.69 (VDD), C104.1
- net VDD_IO_0: now also U102.15 (VDD), C107.1
- net VDD_IO_1: now also U102.41 (VDD), C101.1
- net VDD_IO_2: now also U102.50 (VDD), C108.1
- net VDD_IO_3: now also U102.4 (VDD), C102.1
- net an_0: now also U102.29 (an_0); no longer U101.29 (an_0)
- net an_1: now also U102.30 (an_1); no longer U101.28 (an_1)
- net an_2: now also U101.14 (in_9), U102.31 (an_2); no longer U101.21 (in_4)
- net an_3: now also U101.15 (in_8), U102.34 (an_3); no longer U101.20 (in_5)
- net bidir_0: now also U102.1 (bidir_0)
- net bidir_1: now also U102.2 (bidir_1)
- net bidir_10: now also U102.13 (bidir_10)
- net bidir_11: now also U102.16 (bidir_11)
- net bidir_12: now also U102.17 (bidir_12)
- net bidir_13: now also U102.18 (bidir_13)
- net bidir_14: now also U102.19 (bidir_14)
- net bidir_15: now also U102.20 (bidir_15)
- net bidir_16: now also U102.21 (bidir_16)
- net bidir_17: now also U102.22 (bidir_17)
- net bidir_18: now also U102.25 (bidir_18)
- net bidir_19: now also U102.26 (bidir_19)
- net bidir_2: now also U102.5 (bidir_2)
- net bidir_20: now also U102.27 (bidir_20)
- net bidir_21: now also U102.28 (bidir_21)
- net bidir_22: now also U102.37 (bidir_22)
- net bidir_23: now also U102.38 (bidir_23)
- net bidir_24: now also U102.39 (bidir_24)
- net bidir_25: now also U102.40 (bidir_25)
- net bidir_26: now also U102.43 (bidir_26)
- net bidir_27: now also U102.44 (bidir_27)
- net bidir_28: now also U102.45 (bidir_28)
- net bidir_29: now also U102.46 (bidir_29)
- net bidir_3: now also U102.6 (bidir_3)
- net bidir_30: now also U102.47 (bidir_30)
- net bidir_31: now also U102.48 (bidir_31)
- net bidir_32: now also U102.49 (bidir_32)
- net bidir_33: now also U102.52 (bidir_33)
- net bidir_34: now also U102.53 (bidir_34)
- net bidir_35: now also U102.54 (bidir_35)
- net bidir_36: now also U102.55 (bidir_36)
- net bidir_37: now also U102.56 (bidir_37)
- net bidir_38: now also U102.57 (bidir_38)
- net bidir_39: now also U102.58 (bidir_39)
- net bidir_4: now also U102.7 (bidir_4)
- net bidir_40: now also U101.29 (an_0), U102.59 (bidir_40); no longer U101.17 (in_6)
- net bidir_41: now also U101.28 (an_1), U102.62 (bidir_41); no longer U101.16 (in_7)
- net bidir_42: now also U101.23 (in_2), U102.63 (bidir_42); no longer U101.15 (in_8)
- net bidir_43: now also U101.22 (in_3), U102.64 (bidir_43); no longer U101.14 (in_9)
- net bidir_5: now also U102.8 (bidir_5)
- net bidir_6: now also U102.9 (bidir_6)
- net bidir_7: now also U102.10 (bidir_7)
- net bidir_8: now also U102.11 (bidir_8)
- net bidir_9: now also U102.12 (bidir_9)
- net clk: now also U102.65 (clk)
- net in_0: now also U102.67 (in_0)
- net in_1: now also U102.70 (in_1)
- net in_2: now also U101.17 (in_6), U102.71 (in_2); no longer U101.23 (in_2)
- net in_3: now also U101.16 (in_7), U102.72 (in_3); no longer U101.22 (in_3)
- net rst_n: now also U102.66 (rst_n)
- net an_4: now reaches U102.35 (an_4)
- net an_4: now also U101.20 (in_5)
- net an_5: now reaches U102.36 (an_5)
- net an_5: now also U101.21 (in_4)

Commit message: Diagonal die
Connections:
- net an_0: now also U101.41 (bidir_28); no longer U101.12 (in_11)
- net an_1: now also U101.40 (bidir_29); no longer U101.13 (in_10)
- net an_2: now also U101.39 (bidir_30); no longer U101.14 (in_9)
- net an_3: now also U101.38 (bidir_31); no longer U101.15 (in_8)
- net an_4: now also U101.37 (bidir_32); no longer U101.20 (in_5)
- net an_5: now also U101.36 (bidir_33); no longer U101.21 (in_4)
- net bidir_28: now also U101.35 (bidir_34); no longer U101.41 (bidir_28)
- net bidir_29: now also U101.34 (bidir_35); no longer U101.40 (bidir_29)
- net bidir_30: now also U101.33 (bidir_36); no longer U101.39 (bidir_30)
- net bidir_31: now also U101.32 (bidir_37); no longer U101.38 (bidir_31)
- net bidir_32: now also U101.31 (bidir_38); no longer U101.37 (bidir_32)
- net bidir_33: now also U101.30 (bidir_39); no longer U101.36 (bidir_33)
- net bidir_34: now also U101.29 (an_0); no longer U101.35 (bidir_34)
- net bidir_35: now also U101.28 (an_1); no longer U101.34 (bidir_35)
- net bidir_36: now also U101.23 (in_2); no longer U101.33 (bidir_36)
- net bidir_37: now also U101.22 (in_3); no longer U101.32 (bidir_37)
- net bidir_38: now also U101.21 (in_4); no longer U101.31 (bidir_38)
- net bidir_39: now also U101.20 (in_5); no longer U101.30 (bidir_39)
- net bidir_40: now also U101.17 (in_6); no longer U101.29 (an_0)
- net bidir_41: now also U101.16 (in_7); no longer U101.28 (an_1)
- net bidir_42: now also U101.15 (in_8); no longer U101.23 (in_2)
- net bidir_43: now also U101.14 (in_9); no longer U101.22 (in_3)
- net in_2: now also U101.13 (in_10); no longer U101.17 (in_6)
- net in_3: now also U101.12 (in_11); no longer U101.16 (in_7)
