File: run-1/motherboards/motherboards.kicad_pcb (KiCad board)
At the start: 2 copper layers, 34.6 x 90.2 mm, 8 parts, among them J101 Conn_01x35, J102 Conn_02x35_Counter_Clockwise, J103 Conn_01x35, J104 Conn_01x35, J105 Conn_02x35_Counter_Clockwise, J106 Conn_01x35

Commit message: harmonize maotherboard pin naming
Connections:
- J102 pad 39: Net-(J102-pad_41) -> (no net)
- J103 pad 32: Net-(J102-pad_41) -> Net-(J102-pad_49)
- J105 pad 39: Net-(J105-Pin_39) -> (no net)
- J106 pad 32: Net-(J105-Pin_39) -> Net-(J105-pad_49)
Routing:
- net Net-(J102-pad_49): track 0.00 -> 36.3 mm, vias 0 -> 1
- net Net-(J102-pad_41): track 36.3 -> 0.00 mm, vias 1 -> 0
- net Net-(J105-pad_49): track 0.00 -> 10.4 mm
- net Net-(J105-Pin_39): track 10.4 -> 0.00 mm

Commit message: fix pin numbering on motherboards
Connections:
- J102 pad 39: (no net) -> Net-(J102-pad_49)
- J105 pad 39: (no net) -> Net-(J105-pad_49)
