File: run-1/1x0p5-cob/mezzanine-1x0p5.kicad_pcb (KiCad board)
At the start: 2 copper layers, 14 x 16 mm, 11 parts

Commit message: Update mask
Routing:
- net GND: track 55.3 -> 37.3 mm
Changed lines of the file:
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@@
 		)
 		(fp_rect
-			(start -4.6 -4.7)
-			(end 4.6 4.7)
+			(start -2.1 -1.4)
+			(end 2.1 1.4)
+			(stroke
+				(width 0.1)
+				(type default)
+			)
+			(fill yes)
+			(layer "F.Mask")
+		)
+		(fp_poly
+			(pts
+				(xy -2.9 4.7) (xy 2.4 4.7) (xy 2.4 3.5) (xy -2.4 3.5) (xy -3.4 2.5) (xy -3.4 -2.5) (xy -2.4 -3.5)
+				(xy 2.4 -3.5) (xy 3.4 -2.5) (xy 3.4 2.5) (xy 2.4 3.5) (xy 2.4 4.7) (xy 4.7 4.7) (xy 4.7 -2.9) (xy 2.9 -4.7)
+				(xy -4.7 -4.7) (xy -4.7 2.9)
+			)
 			(stroke
 				(width 0.1)
@@
 		)
 		(fp_circle
-			(center -4.15 4.25)
-			(end -3.75 4.25)
+			(center -4.55 3.85)
+			(end -4.15 3.85)
 			(stroke
 				(width 0)
@@
 			(pinfunction "MP_75")
 			(pintype "power_in")
+			(zone_connect 2)
+			(thermal_bridge_angle 0)
 		)
 		(pad "75" thru_hole circle
@@
 			(pinfunction "MP_75")
 			(pintype "power_in")
+			(zone_connect 2)
+			(thermal_bridge_angle 0)
 		)
 		(pad "75" thru_hole circle
@@
 			(pinfunction "MP_75")
 			(pintype "power_in")
+			(zone_connect 2)
+			(thermal_bridge_angle 0)
 		)
 		(pad "75" smd roundrect
@@
 			(pinfunction "MP_75")
 			(pintype "power_in")
+			(zone_connect 2)
+			(thermal_bridge_angle 0)
 		)
 		(pad "75" thru_hole circle
@@
 			(pinfunction "MP_75")
 			(pintype "power_in")
+			(zone_connect 2)
+			(thermal_bridge_angle 0)
 		)
 		(pad "75" thru_hole circle
@@
 			(pinfunction "MP_75")
 			(pintype "power_in")
+			(zone_connect 2)
+			(thermal_bridge_angle 0)
 		)
 		(embedded_fonts no)
@@
 		)
 		(embedded_fonts no)
-		(model "${KICAD6_3DMODEL_DIR}/Capacitor_SMD.3dshapes/C_0201_0603Metric.wrl"
+		(model "${KICAD10_3DMODEL_DIR}/Capacitor_SMD.3dshapes/C_0201_0603Metric.step"
 			(offset
 				(xyz 0 0 0)
@@
 		)
 		(embedded_fonts no)
-		(model "${KICAD6_3DMODEL_DIR}/Capacitor_SMD.3dshapes/C_0201_0603Metric.wrl"
+		(model "${KICAD10_3DMODEL_DIR}/Capacitor_SMD.3dshapes/C_0201_0603Metric.step"
 			(offset
 				(xyz 0 0 0)
@@
 		)
 		(embedded_fonts no)
-		(model "${KICAD6_3DMODEL_DIR}/Capacitor_SMD.3dshapes/C_0201_0603Metric.wrl"
+		(model "${KICAD10_3DMODEL_DIR}/Capacitor_SMD.3dshapes/C_0201_0603Metric.step"
 			(offset
 				(xyz 0 0 0)
@@
 		)
 		(embedded_fonts no)
-		(model "${KICAD6_3DMODEL_DIR}/Capacitor_SMD.3dshapes/C_0201_0603Metric.wrl"
+		(model "${KICAD10_3DMODEL_DIR}/Capacitor_SMD.3dshapes/C_0201_0603Metric.step"
 			(offset
 				(xyz 0 0 0)
@@
 		)
 		(embedded_fonts no)
-		(model "${KICAD6_3DMODEL_DIR}/Capacitor_SMD.3dshapes/C_0201_0603Metric.wrl"
+		(model "${KICAD10_3DMODEL_DIR}/Capacitor_SMD.3dshapes/C_0201_0603Metric.step"
 			(offset
 				(xyz 0 0 0)
@@
 		)
 		(embedded_fonts no)
-		(model "${KICAD6_3DMODEL_DIR}/Capacitor_SMD.3dshapes/C_0201_0603Metric.wrl"
+		(model "${KICAD10_3DMODEL_DIR}/Capacitor_SMD.3dshapes/C_0201_0603Metric.step"
 			(offset
 				(xyz 0 0 0)
@@
 		)
 		(embedded_fonts no)
-		(model "${KICAD6_3DMODEL_DIR}/Capacitor_SMD.3dshapes/C_0201_0603Metric.wrl"
+		(model "${KICAD10_3DMODEL_DIR}/Capacitor_SMD.3dshapes/C_0201_0603Metric.step"
 			(offset
 				(xyz 0 0 0)
@@
 		)
 		(embedded_fonts no)
-		(model "${KICAD6_3DMODEL_DIR}/Capacitor_SMD.3dshapes/C_0201_0603Metric.wrl"
+		(model "${KICAD10_3DMODEL_DIR}/Capacitor_SMD.3dshapes/C_0201_0603Metric.step"
 			(offset
 				(xyz 0 0 0)
@@
 	)
 	(segment
-		(start 143.37 93.635)
-		(end 143.37 89.635)
-		(width 0.4)
-		(layer "F.Cu")
-		(net "GND")
-	)
-	(segment
 		(start 143.95 86.05)
 		(end 143.95 85.3)
@@
 	)
 	(segment
-		(start 138.32 89.635)
-		(end 138.32 93.585)
-		(width 0.4)
-		(layer "F.Cu")
-		(net "GND")
-	)
-	(segment
 		(start 138.920001 95.784998)
 		(end 138.920001 96.429999)
@@
 	)
 	(segment
-		(start 138.96 93.635)
-		(end 143.37 93.635)
-		(width 0.4)
-		(layer "F.Cu")
-		(net "GND")
-	)
-	(segment
 		(start 137.79 97.84)
 		(end 137.43 98.2)
@@
 	)
 	(segment
-		(start 138.95 89.635)
-		(end 138.32 89.635)
-		(width 0.4)
-		(layer "F.Cu")
-		(net "GND")
-	)
-	(segment
-		(start 138.37 93.635)
-		(end 138.96 93.635)
-		(width 0.4)
-		(layer "F.Cu")
-		(net "GND")
-	)
-	(segment
 		(start 143.12 89.385)
 		(end 143.37 89.635)
@@
 	)
 	(segment
-		(start 143.37 89.635)
-		(end 138.95 89.635)
-		(width 0.4)
-		(layer "F.Cu")
-		(net "GND")
-	)
-	(segment
 		(start 138.32 93.585)
 		(end 138.37 93.635)
@@
 		(polygon
 			(pts
-				(xy 136.1 86.725) (xy 145.65 86.725) (xy 145.65 96.525) (xy 136.1 96.525)
+				(xy 136.05 86.825) (xy 136.9 86.825) (xy 136.9 87.75) (xy 136.05 87.75)
+			)
+		)
+	)
+	(zone
+		(layer "F.Cu")
+		(hatch edge 0.5)
+		(connect_pads
+			(clearance 0)
+		)
+		(min_thickness 0.15)
+		(keepout
+			(tracks allowed)
+			(vias allowed)
+			(pads allowed)
+			(copperpour not_allowed)
+			(footprints allowed)
+		)
+		(placement
+			(enabled no)
+			(sheetname "/")
+		)
+		(fill
+			(thermal_gap 0.5)
+			(thermal_bridge_width 0.5)
+			(island_removal_mode 1)
+		)
+		(polygon
+			(pts
+				(xy 144.8 95.6) (xy 145.65 95.6) (xy 145.65 96.525) (xy 144.8 96.525)
 			)
 		)
