File: run-1/0p5x1-cob/mezzanine-0p5x1.kicad_sch (KiCad schematic)
At the start: 10 parts

Commit message: Check symbols against template pad frame
Connections:
- net GND: now also U102.33 (GND), U102.48 (GND); no longer U102.31 (GND), U102.50 (GND)
- net VDD_CORE_0: now also U102.34 (VDD); no longer U102.32 (VDD)
- net VDD_IO_2: now also U102.47 (VDD); no longer U102.49 (VDD)
- net bidir_18: now also U102.31 (bidir_18); no longer U102.33 (bidir_18)
- net bidir_19: now also U102.32 (bidir_19); no longer U102.34 (bidir_19)
- net bidir_24: now also U102.49 (bidir_24); no longer U102.47 (bidir_24)
- net bidir_25: now also U102.50 (bidir_25); no longer U102.48 (bidir_25)
Changed lines of the file:
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@@
 	)
 	(junction
-		(at 247.65 101.6)
-		(diameter 0)
-		(color 0 0 0 0)
-	)
-	(junction
-		(at 160.02 101.6)
+		(at 160.02 106.68)
 		(diameter 0)
 		(color 0 0 0 0)
@@
 		(color 0 0 0 0)
 	)
+	(junction
+		(at 247.65 106.68)
+		(diameter 0)
+		(color 0 0 0 0)
+	)
+	(wire
+		(pts
+			(xy 160.02 106.68) (xy 160.02 121.92)
+		)
+		(stroke
+			(width 0)
+			(type default)
+		)
+	)
 	(wire
 		(pts
@@
 	(wire
 		(pts
-			(xy 160.02 101.6) (xy 179.07 101.6)
-		)
-		(stroke
-			(width 0)
-			(type default)
-		)
-	)
-	(wire
-		(pts
-			(xy 227.33 101.6) (xy 247.65 101.6)
-		)
-		(stroke
-			(width 0)
-			(type default)
-		)
-	)
-	(wire
-		(pts
 			(xy 110.49 80.01) (xy 110.49 100.33)
 		)
@@
 	(wire
 		(pts
-			(xy 247.65 78.74) (xy 247.65 101.6)
+			(xy 247.65 78.74) (xy 247.65 106.68)
 		)
 		(stroke
@@
 	(wire
 		(pts
-			(xy 160.02 78.74) (xy 160.02 101.6)
+			(xy 160.02 78.74) (xy 160.02 106.68)
 		)
 		(stroke
@@
 	(wire
 		(pts
+			(xy 227.33 106.68) (xy 247.65 106.68)
+		)
+		(stroke
+			(width 0)
+			(type default)
+		)
+	)
+	(wire
+		(pts
 			(xy 227.33 78.74) (xy 247.65 78.74)
 		)
@@
 	(wire
 		(pts
-			(xy 160.02 101.6) (xy 160.02 121.92)
-		)
-		(stroke
-			(width 0)
-			(type default)
-		)
-	)
-	(wire
-		(pts
 			(xy 40.64 97.79) (xy 54.61 97.79)
 		)
@@
 	(wire
 		(pts
-			(xy 247.65 101.6) (xy 247.65 138.43)
-		)
-		(stroke
-			(width 0)
-			(type default)
-		)
-	)
-	(wire
-		(pts
 			(xy 40.64 97.79) (xy 40.64 137.16)
 		)
@@
 	(wire
 		(pts
+			(xy 160.02 106.68) (xy 179.07 106.68)
+		)
+		(stroke
+			(width 0)
+			(type default)
+		)
+	)
+	(wire
+		(pts
 			(xy 110.49 59.69) (xy 110.49 80.01)
+		)
+		(stroke
+			(width 0)
+			(type default)
+		)
+	)
+	(wire
+		(pts
+			(xy 247.65 106.68) (xy 247.65 138.43)
 		)
 		(stroke
@@
 		)
 	)
+	(label "bidir_24"
+		(at 227.33 104.14 0)
+		(effects
+			(font
+				(size 1.27 1.27)
+			)
+			(justify left bottom)
+		)
+	)
 	(label "VDD_IO_3"
 		(at 201.93 33.02 90)
@@
 		)
 	)
-	(label "VDD_CORE_0"
-		(at 179.07 104.14 180)
-		(effects
-			(font
-				(size 1.27 1.27)
-			)
-			(justify right bottom)
-		)
-	)
 	(label "bidir_23"
 		(at 227.33 111.76 0)
@@
 		)
 	)
+	(label "bidir_19"
+		(at 179.07 104.14 180)
+		(effects
+			(font
+				(size 1.27 1.27)
+			)
+			(justify right bottom)
+		)
+	)
 	(label "an_3"
 		(at 207.01 127 270)
@@
 		)
 	)
-	(label "bidir_25"
-		(at 227.33 106.68 0)
-		(effects
-			(font
-				(size 1.27 1.27)
-			)
-			(justify left bottom)
-		)
-	)
 	(label "bidir_42"
 		(at 227.33 48.26 0)
@@
 		)
 	)
-	(label "VDD_IO_2"
-		(at 227.33 104.14 0)
-		(effects
-			(font
-				(size 1.27 1.27)
-			)
-			(justify left bottom)
-		)
-	)
 	(label "PWR_AUX_0"
 		(at 92.71 77.47 0)
@@
 		)
 	)
-	(label "bidir_18"
-		(at 179.07 106.68 180)
-		(effects
-			(font
-				(size 1.27 1.27)
-			)
-			(justify right bottom)
-		)
-	)
 	(label "bidir_29"
 		(at 54.61 110.49 180)
@@
 		)
 	)
+	(label "VDD_CORE_0"
+		(at 179.07 109.22 180)
+		(effects
+			(font
+				(size 1.27 1.27)
+			)
+			(justify right bottom)
+		)
+	)
 	(label "bidir_14"
 		(at 92.71 72.39 0)
@@
 		)
 	)
+	(label "bidir_25"
+		(at 227.33 101.6 0)
+		(effects
+			(font
+				(size 1.27 1.27)
+			)
+			(justify left bottom)
+		)
+	)
 	(label "bidir_3"
 		(at 92.71 39.37 0)
@@
 		)
 	)
-	(label "bidir_24"
-		(at 227.33 109.22 0)
-		(effects
-			(font
-				(size 1.27 1.27)
-			)
-			(justify left bottom)
-		)
-	)
 	(label "PWR_AUX_1"
 		(at 227.33 81.28 0)
@@
 		)
 	)
+	(label "VDD_IO_2"
+		(at 227.33 109.22 0)
+		(effects
+			(font
+				(size 1.27 1.27)
+			)
+			(justify left bottom)
+		)
+	)
 	(label "bidir_20"
 		(at 92.71 92.71 0)
@@
 		)
 	)
-	(label "bidir_19"
-		(at 179.07 109.22 180)
-		(effects
-			(font
+	(label "bidir_18"
+		(at 179.07 101.6 180)
+		(effects
+			(font
