File: run-1/tqva-cob/tqva-cob.kicad_sch (KiCad schematic)
At the start: 6 parts

Commit message: TQVA CoB, tweaks
Connections:
- net bidir_27: now also U101.42 (bidir_27); no longer U101.26 (in_1)
- net bidir_28: now also U101.41 (bidir_28); no longer U101.23 (in_2)
- net bidir_29: now also U101.40 (bidir_29); no longer U101.22 (in_3)
- net bidir_30: now also U101.39 (bidir_30); no longer U101.21 (in_4)
- net bidir_31: now also U101.38 (bidir_31); no longer U101.20 (in_5)
- net bidir_32: now also U101.37 (bidir_32); no longer U101.17 (in_6)
- net in_0: now also U101.12 (in_11); no longer U101.30 (bidir_39)
- net in_1: now also U101.13 (in_10); no longer U101.29 (an_0)
- net an_0: no longer names the net of U102.34 (an_0)
- net an_0: no longer U101.42 (bidir_27)
- net an_1: no longer names the net of U102.35 (an_1)
- net an_1: no longer U101.41 (bidir_28)
- net an_2: no longer names the net of U102.38 (an_2)
- net an_2: no longer U101.40 (bidir_29)
- net an_3: no longer names the net of U102.39 (an_3)
- net an_3: no longer U101.31 (bidir_38)
- net bidir_33: no longer names the net of U102.52 (bidir_33)
- net bidir_33: no longer U101.16 (in_7)
- net bidir_34: no longer names the net of U102.53 (bidir_34)
- net bidir_34: no longer U101.15 (in_8)
- net bidir_35: no longer names the net of U102.54 (bidir_35)
- net bidir_35: no longer U101.14 (in_9)
- net bidir_36: no longer names the net of U102.55 (bidir_36)
- net bidir_36: no longer U101.13 (in_10)
- net bidir_37: no longer names the net of U102.56 (bidir_37)
- net bidir_37: no longer U101.12 (in_11)
- net in_2: no longer names the net of U102.44 (in_2)
- net in_2: no longer U101.28 (an_1)
- net in_3: no longer names the net of U102.45 (in_3)
- net in_3: no longer U101.27 (in_0)
- no-connect marks 10 -> 32
Other:
- company: (none) -> Team Rebellion
- title: (none) -> Wafer Space TQVA CoB

Commit message: Check symbols against template pad frame
Parts:
- U102: symbol WaferSpace:0p5x0p5 -> WaferSpace:tqva
Changed lines of the file:
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@@
 	)
 	(symbol
-		(lib_id "WaferSpace:0p5x0p5")
+		(lib_id "WaferSpace:tqva")
 		(at 179.07 99.06 0)
 		(unit 1)
